File: documentatie/bronnen/Electric-Sceme/CNC3DPrinter/CNC3DFull/CNC3DFull.kicad_sch (KiCad schematic)
At the start: 11 parts, among them M2 Stepper_Motor_bipolar, M3 Stepper_Motor_bipolar, M5 Stepper_Motor_bipolar, U2 ATmega2560-16A

Commit message: .
Connections:
- net XDirPin: now also U2.78 (PA0)
- net XStepPin: now also U2.77 (PA1)
- net YDirPin: now also U2.76 (PA2)
- net YStepPin: now also U2.75 (PA3)
- net ZDirPin: now also U2.74 (PA4)
- net ZStepPin: now also U2.73 (PA5)
- net at U2.43 (PD0): now also EncoderX. (Vin)
- net at U2.44 (PD1): now also EncoderX. (Vin)
- net at U2.45 (PD2): now also EncoderY. (Vin)
- net at U2.46 (PD3): now also EncoderY. (Vin)
- net at U2.6 (PE4): now also EncoderZ. (Vin)
- net at U2.7 (PE5): now also EncoderZ. (Vin)
Other:
- company: (none) -> Sens2Sea
- title: (none) -> CNC 3 assen motor aansturing
Changed lines of the file:
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@@
 (kicad_sch (version 20230121) (generator eeschema)
   (paper "A4")
+  (title_block
+    (title "CNC 3 assen motor aansturing")
+    (date "2026-01-08")
+    (rev "2026-01-08")
+    (company "Sens2Sea")
+  )
   (junction (at 237.49 30.48) (diameter 0) (color 0 0 0 0)
   )
@@
     (stroke (width 0) (type default))
   )
+  (wire (pts (xy 96.52 114.3) (xy 96.52 115.57))
+    (stroke (width 0) (type default))
+  )
+  (wire (pts (xy 110.49 138.43) (xy 153.67 138.43))
+    (stroke (width 0) (type default))
+  )
   (wire (pts (xy 105.41 39.37) (xy 105.41 24.13))
     (stroke (width 0) (type default))
@@
     (stroke (width 0) (type default))
   )
+  (wire (pts (xy 96.52 114.3) (xy 153.67 114.3))
+    (stroke (width 0) (type default))
+  )
   (wire (pts (xy 212.09 43.18) (xy 212.09 40.64))
     (stroke (width 0) (type default))
@@
     (stroke (width 0) (type default))
   )
+  (wire (pts (xy 93.98 85.09) (xy 153.67 85.09))
+    (stroke (width 0) (type default))
+  )
   (wire (pts (xy 111.76 31.75) (xy 113.03 31.75))
     (stroke (width 0) (type default))
@@
     (stroke (width 0) (type default))
   )
+  (wire (pts (xy 93.98 111.76) (xy 153.67 111.76))
+    (stroke (width 0) (type default))
+  )
   (wire (pts (xy 143.51 33.02) (xy 140.97 33.02))
     (stroke (width 0) (type default))
   )
+  (wire (pts (xy 83.82 143.51) (xy 113.03 143.51))
+    (stroke (width 0) (type default))
+  )
   (wire (pts (xy 165.1 35.56) (xy 168.91 35.56))
     (stroke (width 0) (type default))
@@
     (stroke (width 0) (type default))
   )
-  (wire (pts (xy 153.67 111.76) (xy 152.4 111.76))
-    (stroke (width 0) (type default))
-  )
   (wire (pts (xy 237.49 30.48) (xy 240.03 30.48))
     (stroke (width 0) (type default))
   )
-  (wire (pts (xy 153.67 114.3) (xy 149.86 114.3))
-    (stroke (width 0) (type default))
-  )
   (wire (pts (xy 252.73 58.42) (xy 252.73 72.39))
     (stroke (width 0) (type default))
@@
     (stroke (width 0) (type default))
   )
+  (wire (pts (xy 93.98 113.03) (xy 83.82 113.03))
+    (stroke (width 0) (type default))
+  )
   (wire (pts (xy 140.97 29.21) (xy 140.97 30.48))
     (stroke (width 0) (type default))
   )
-  (wire (pts (xy 153.67 87.63) (xy 149.86 87.63))
+  (wire (pts (xy 96.52 87.63) (xy 153.67 87.63))
     (stroke (width 0) (type default))
   )
@@
     (stroke (width 0) (type default))
   )
+  (wire (pts (xy 93.98 111.76) (xy 93.98 113.03))
+    (stroke (width 0) (type default))
+  )
   (wire (pts (xy 111.76 24.13) (xy 111.76 31.75))
     (stroke (width 0) (type default))
@@
     (stroke (width 0) (type default))
   )
+  (wire (pts (xy 93.98 85.09) (xy 93.98 107.95))
+    (stroke (width 0) (type default))
+  )
   (wire (pts (xy 163.83 33.02) (xy 173.99 33.02))
     (stroke (width 0) (type default))
   )
+  (wire (pts (xy 110.49 140.97) (xy 83.82 140.97))
+    (stroke (width 0) (type default))
+  )
   (wire (pts (xy 191.77 38.1) (xy 185.42 38.1))
     (stroke (width 0) (type default))
@@
     (stroke (width 0) (type default))
   )
+  (wire (pts (xy 93.98 107.95) (xy 83.82 107.95))
+    (stroke (width 0) (type default))
+  )
   (wire (pts (xy 173.99 33.02) (xy 173.99 35.56))
     (stroke (width 0) (type default))
@@
     (stroke (width 0) (type default))
   )
+  (wire (pts (xy 110.49 138.43) (xy 110.49 140.97))
+    (stroke (width 0) (type default))
+  )
   (wire (pts (xy 21.59 26.67) (xy 21.59 22.86))
     (stroke (width 0) (type default))
   )
+  (wire (pts (xy 96.52 87.63) (xy 96.52 110.49))
+    (stroke (width 0) (type default))
+  )
   (wire (pts (xy 212.09 33.02) (xy 222.25 33.02))
     (stroke (width 0) (type default))
@@
     (stroke (width 0) (type default))
   )
-  (wire (pts (xy 153.67 85.09) (xy 152.4 85.09))
+  (wire (pts (xy 96.52 115.57) (xy 83.82 115.57))
     (stroke (width 0) (type default))
   )
@@
     (stroke (width 0) (type default))
   )
-  (wire (pts (xy 153.67 138.43) (xy 152.4 138.43))
+  (wire (pts (xy 96.52 110.49) (xy 83.82 110.49))
     (stroke (width 0) (type default))
   )
@@
     (stroke (width 0) (type default))
   )
-  (wire (pts (xy 153.67 140.97) (xy 149.86 140.97))
+  (wire (pts (xy 113.03 140.97) (xy 113.03 143.51))
+    (stroke (width 0) (type default))
+  )
+  (wire (pts (xy 113.03 140.97) (xy 153.67 140.97))
     (stroke (width 0) (type default))
   )
@@
     )
   )
+  (global_label "ZDirPin" (shape input) (at 83.82 49.53 0) (fields_autoplaced)
+    (effects (font (size 1.27 1.27)) (justify left))
+    (property "Intersheetrefs" "${INTERSHEET_REFS}" (at 93.6995 49.53 0)
+      (effects (font (size 1.27 1.27)) (justify left) hide)
+    )
+  )
   (global_label "Logic 5v" (shape input) (at 27.94 26.67 270) (fields_autoplaced)
     (effects (font (size 1.27 1.27)) (justify right))
@@
     )
   )
+  (global_label "ZStepPin" (shape input) (at 83.82 52.07 0) (fields_autoplaced)
+    (effects (font (size 1.27 1.27)) (justify left))
+    (property "Intersheetrefs" "${INTERSHEET_REFS}" (at 95.2113 52.07 0)
+      (effects (font (size 1.27 1.27)) (justify left) hide)
+    )
+  )
   (global_label "Logic 5V" (shape input) (at 166.37 87.63 0) (fields_autoplaced)
     (effects (font (size 1.27 1.27)) (justify left))
@@
     )
   )
+  (global_label "YStepPin" (shape input) (at 83.82 46.99 0) (fields_autoplaced)
+    (effects (font (size 1.27 1.27)) (justify left))
+    (property "Intersheetrefs" "${INTERSHEET_REFS}" (at 95.0904 46.99 0)
+      (effects (font (size 1.27 1.27)) (justify left) hide)
+    )
+  )
+  (global_label "XStepPin" (shape input) (at 83.82 41.91 0) (fields_autoplaced)
+    (effects (font (size 1.27 1.27)) (justify left))
+    (property "Intersheetrefs" "${INTERSHEET_REFS}" (at 95.2113 41.91 0)
+      (effects (font (size 1.27 1.27)) (justify left) hide)
+    )
+  )
   (global_label "XDirPin" (shape input) (at 240.03 43.18 180) (fields_autoplaced)
     (effects (font (size 1.27 1.27)) (justify right))
@@
     )
   )
+  (global_label "XDirPin" (shape input) (at 83.82 39.37 0) (fields_autoplaced)
+    (effects (font (size 1.27 1.27)) (justify left))
+    (property "Intersheetrefs" "${INTERSHEET_REFS}" (at 93.6995 39.37 0)
+      (effects (font (size 1.27 1.27)) (justify left) hide)
+    )
+  )
   (global_label "Logic 5V" (shape input) (at 166.37 114.3 0) (fields_autoplaced)
     (effects (font (size 1.27 1.27)) (justify left))
@@
     )
   )
+  (global_label "YDirPin" (shape input) (at 83.82 44.45 0) (fields_autoplaced)
+    (effects (font (size 1.27 1.27)) (justify left))
+    (property "Intersheetrefs" "${INTERSHEET_REFS}" (at 93.5786 44.45 0)
+      (effects (font (size 1.27 1.27)) (justify left) hide)
+    )
+  )

Commit message: .
Parts:
- added M1: Stepper_Motor_bipolar, symbol Motor:Stepper_Motor_bipolar
- added XStepper-2: Pololu_Breakout_DRV8825, Module:Pololu_Breakout-16_15.2x20.3mm, symbol Driver_Motor:Pololu_Breakout_DRV8825
- renumbered XStepper to XStepper-1
Connections:
- net +12V: now also XStepper-2.8 (VMOT)
- net GND1: now also XStepper-2.1 (GND), XStepper-2.7 (GND), XStepper-2.9 (~{EN})
- net Logic 5V: now also XStepper-2.13 (~{RST}), XStepper-2.14 (~{SLP})
- net XDirPin: now also XStepper-2.16 (DIR)
- net XStepPin: now also XStepper-2.15 (STEP)
- new net: M1.1, XStepper-2.3 (A2)
- new net: M1.2 (-), XStepper-2.4 (A1)
- new net: M1.3, XStepper-2.5 (B1)
- new net: M1.4, XStepper-2.6 (B2)

Commit message: opleverset aangemaakt, stageverslag verbeterd
Parts:
- removed M1: Stepper_Motor_bipolar, symbol Motor:Stepper_Motor_bipolar
- removed XStepper-2: Pololu_Breakout_DRV8825, Module:Pololu_Breakout-16_15.2x20.3mm, symbol Driver_Motor:Pololu_Breakout_DRV8825
- added C1, C3: capacitor 100 μf, symbol Device:C_Polarized_US
Connections:
- net +12V: now also C1.1, C3.1
- net GND1: now also C1.2, C3.2
Other:
- moved on the sheet: M3, M5, YStepper, ZStepper
